Commit message: fix a bug in urdf file( wrong direction for rotation angle)

File: urdf/cassie.urdf (robot description, URDF)
Before this commit: robot cassie, 17 links, 16 joints
Joints:
- joint hip_rotation_left: axis 1 0 0 -> -1 0 0
- joint hip_rotation_right: axis 1 0 0 -> -1 0 0

File: urdf/cassie.xacro (robot description, xacro)
@@ -248,5 +248,5 @@
     <joint name="hip_rotation_${side}" type="continuous">
       <origin xyz="0 0 -0.09" rpy="0 ${pi/2} ${-pi/2}"/>
-      <axis xyz="1 0 0"/>
+      <axis xyz="-1 0 0"/>
       <parent link="${side}_pelvis_rotation" />
       <child link="${side}_hip" />
